Commit message: feat: can load ro arm m2 s but it's stupid

File: src/amr_descriptions/model/roarm_description/urdf/roarm.urdf.xacro (robot description, xacro)
@@ -2,4 +2,6 @@
 <robot
   name="roarm_description">
+  <!-- Dummy link to fix KDL root inertia warning -->
+  <link name="base_footprint"/>
   <link
     name="base_link">
@@ -24,22 +26,27 @@
       <geometry>
         <mesh
-          filename="package://roarm_description/meshes/base_link.STL" />
-      </geometry>
-      <material
-        name="">
-        <color
-          rgba="0.752941176470588 0.752941176470588 0.752941176470588 1" />
-      </material>
-    </visual>
-    <collision>
-      <origin
-        xyz="0 0 0"
-        rpy="0 0 0" />
-      <geometry>
-        <mesh
-          filename="package://roarm_description/meshes/base_link.STL" />
-      </geometry>
-    </collision>
-  </link>
+          filename="package://amr_descriptions/model/roarm_description/meshes/base_link.STL" />
+      </geometry>
+      <material
+        name="">
+        <color
+          rgba="0.752941176470588 0.752941176470588 0.752941176470588 1" />
+      </material>
+    </visual>
+    <collision>
+      <origin
+        xyz="0 0 0"
+        rpy="0 0 0" />
+      <geometry>
+        <mesh
+          filename="package://amr_descriptions/model/roarm_description/meshes/base_link.STL" />
+      </geometry>
+    </collision>
+  </link>
+  <joint name="base_footprint_to_base_link" type="fixed">
+    <parent link="base_footprint"/>
+    <child link="base_link"/>
+    <origin xyz="0 0 0" rpy="0 0 0"/>
+  </joint>
   <link
     name="link1">
@@ -64,19 +71,19 @@
       <geometry>
         <mesh
-          filename="package://roarm_description/meshes/link1.STL" />
-      </geometry>
-      <material
-        name="">
-        <color
-          rgba="0.752941176470588 0.752941176470588 0.752941176470588 1" />
-      </material>
-    </visual>
-    <collision>
-      <origin
-        xyz="0 0 0"
-        rpy="0 0 0" />
-      <geometry>
-        <mesh
-          filename="package://roarm_description/meshes/link1.STL" />
+          filename="package://amr_descriptions/model/roarm_description/meshes/link1.STL" />
+      </geometry>
+      <material
+        name="">
+        <color
+          rgba="0.752941176470588 0.752941176470588 0.752941176470588 1" />
+      </material>
+    </visual>
+    <collision>
+      <origin
+        xyz="0 0 0"
+        rpy="0 0 0" />
+      <geometry>
+        <mesh
+          filename="package://amr_descriptions/model/roarm_description/meshes/link1.STL" />
       </geometry>
     </collision>
@@ -122,19 +129,19 @@
       <geometry>
         <mesh
-          filename="package://roarm_description/meshes/link2.STL" />
-      </geometry>
-      <material
-        name="">
-        <color
-          rgba="0.752941176470588 0.752941176470588 0.752941176470588 1" />
-      </material>
-    </visual>
-    <collision>
-      <origin
-        xyz="0 0 0"
-        rpy="0 0 0" />
-      <geometry>
-        <mesh
-          filename="package://roarm_description/meshes/link2.STL" />
+          filename="package://amr_descriptions/model/roarm_description/meshes/link2.STL" />
+      </geometry>
+      <material
+        name="">
+        <color
+          rgba="0.752941176470588 0.752941176470588 0.752941176470588 1" />
+      </material>
+    </visual>
+    <collision>
+      <origin
+        xyz="0 0 0"
+        rpy="0 0 0" />
+      <geometry>
+        <mesh
+          filename="package://amr_descriptions/model/roarm_description/meshes/link2.STL" />
       </geometry>
     </collision>
@@ -180,19 +187,19 @@
       <geometry>
         <mesh
-          filename="package://roarm_description/meshes/link3.STL" />
-      </geometry>
-      <material
-        name="">
-        <color
-          rgba="0.752941176470588 0.752941176470588 0.752941176470588 1" />
-      </material>
-    </visual>
-    <collision>
-      <origin
-        xyz="0 0 0"
-        rpy="0 0 0" />
-      <geometry>
-        <mesh
-          filename="package://roarm_description/meshes/link3.STL" />
+          filename="package://amr_descriptions/model/roarm_description/meshes/link3.STL" />
+      </geometry>
+      <material
+        name="">
+        <color
+          rgba="0.752941176470588 0.752941176470588 0.752941176470588 1" />
+      </material>
+    </visual>
+    <collision>
+      <origin
+        xyz="0 0 0"
+        rpy="0 0 0" />
+      <geometry>
+        <mesh
+          filename="package://amr_descriptions/model/roarm_description/meshes/link3.STL" />
       </geometry>
     </collision>
@@ -238,5 +245,5 @@
       <geometry>
         <mesh
-          filename="package://roarm_description/meshes/gripper_link.STL" />
+          filename="package://amr_descriptions/model/roarm_description/meshes/gripper_link.STL" />
       </geometry>
       <material
@@ -252,5 +259,5 @@
       <geometry>
         <mesh
-          filename="package://roarm_description/meshes/gripper_link.STL" />
+          filename="package://amr_descriptions/model/roarm_description/meshes/gripper_link.STL" />
       </geometry>
     </collision>

File: src/amr_descriptions/model/roarm_description/urdf/roarm.xacro (robot description, xacro)
@@ -2,8 +2,8 @@
 <robot name="roarm" xmlns:xacro="http://www.ros.org/wiki/xacro">
     <!-- Include URDF description -->
-    <xacro:include filename="$(find roarm_description)/urdf/roarm.urdf.xacro"/>
+    <xacro:include filename="$(find amr_descriptions)/model/roarm_description/urdf/roarm.urdf.xacro"/>
     <!-- Include Gazebo plugins -->
-    <xacro:include filename="$(find roarm_description)/urdf/roarm_gazebo.xacro"/>
+    <xacro:include filename="$(find amr_descriptions)/model/roarm_description/urdf/roarm_gazebo.xacro"/>
     <!-- Include ros2_control -->
-    <xacro:include filename="$(find roarm_description)/urdf/roarm_ros2_control.xacro"/>
+    <xacro:include filename="$(find amr_descriptions)/model/roarm_description/urdf/roarm_ros2_control.xacro"/>
 </robot>

File: src/amr_descriptions/model/roarm_description/urdf/roarm_gazebo.xacro (robot description, xacro)
@@ -3,6 +3,6 @@
   <!-- Gazebo plugin for ros2_control (Ignition Gazebo) -->
   <gazebo>
-    <plugin filename="ign_ros2_control-system" name="ign_ros2_control::IgnitionROS2ControlPlugin">
-      <parameters>$(find roarm_description)/config/roarm_controllers.yaml</parameters>
+    <plugin filename="gz_ros2_control-system" name="gz_ros2_control::GazeboSimROS2ControlPlugin">
+      <parameters>$(find amr_descriptions)/model/roarm_description/config/ros2_controller.yaml</parameters>
     </plugin>
   </gazebo>
