Commit message: feat: add zed2 in gazebo but dont have wheels

File: src/amr_descriptions/model/human/model.urdf (robot description, URDF)
Before this commit: robot human, 14 links, 13 joints
Links:
- added link left_hand, mass 0.3; collision sphere radius=0.04; visual sphere radius=0.04
- added link right_hand, mass 0.3; collision sphere radius=0.04; visual sphere radius=0.04
Joints:
- added joint left_wrist_joint: type fixed, parent left_forearm, child left_hand, origin xyz=0 0 -0.18 rpy=0 0 0
- added joint right_wrist_joint: type fixed, parent right_forearm, child right_hand, origin xyz=0 0 -0.18 rpy=0 0 0
