Commit message: feat: push guide for MPC

File: src/amr_descriptions/model/wheeled/urdf/mobile_robot.xacro (robot description, xacro)
@@ -350,10 +350,4 @@
             <material name="black"/>
         </visual>
-        <collision>
-            <origin xyz="0.0 0.0 0.0" rpy="0.0 0.0 0.0"/>
-            <geometry>
-                <cylinder radius="0.04" length="0.03"/>
-            </geometry>
-        </collision>
         <inertial>
             <origin xyz="0.0 0.0 0.0" rpy="0.0 0.0 0.0"/>
