Commit message: feat: can't control with teleop

File: src/amr_descriptions/model/wheeled/urdf/gazebo.xacro (robot description, xacro)
@@ -149,6 +149,4 @@
     </camera>
     <noise><type>gaussian</type><mean>0.0</mean><stddev>0.003</stddev></noise>
-    <plugin filename="ignition-gazebo-camera-system"
-            name="ignition::gazebo::systems::Camera"/>
   </sensor>
 </gazebo>
@@ -173,7 +171,45 @@
     </camera>
     <noise><type>gaussian</type><mean>0.0</mean><stddev>0.003</stddev></noise>
-    <plugin filename="ignition-gazebo-camera-system"
-            name="ignition::gazebo::systems::Camera"/>
   </sensor>
 </gazebo>
+  <!-- ============================================ -->
+  <!-- ROS2 CONTROL CONFIGURATION -->
+  <!-- ============================================ -->
+  <ros2_control name="GazeboSystem" type="system">
+    <hardware>
+      <plugin>gz_ros2_control/GazeboSimSystem</plugin>
+    </hardware>
+    <joint name="left_wheel_joint">
+      <command_interface name="velocity">
+        <param name="min">-10</param>
+        <param name="max">10</param>
+      </command_interface>
+      <state_interface name="velocity"/>
+      <state_interface name="position"/>
+    </joint>
+    <joint name="right_wheel_joint">
+      <command_interface name="velocity">
+        <param name="min">-10</param>
+        <param name="max">10</param>
+      </command_interface>
+      <state_interface name="velocity"/>
+      <state_interface name="position"/>
+    </joint>
+  </ros2_control>
+  <!-- ============================================ -->
+  <!-- GAZEBO PLUGINS -->
+  <!-- ============================================ -->
+  <gazebo>
+    <!-- ros2_control plugin -->
+    <plugin filename="gz_ros2_control-system" name="gz_ros2_control::GazeboSimROS2ControlPlugin">
+      <parameters>$(find amr_descriptions)/model/wheeled/config/ros2_control.yaml</parameters>
+    </plugin>
+    <!-- IMU system -->
+    <plugin filename="gz-sim-imu-system" name="gz::sim::systems::Imu">
+    </plugin>
+    <!-- Sensors system for camera -->
+    <plugin filename="gz-sim-sensors-system" name="gz::sim::systems::Sensors">
+      <render_engine>ogre2</render_engine>
+    </plugin>
+  </gazebo>
 </robot>

File: src/amr_descriptions/model/wheeled/urdf/mobile_robot.urdf.xacro (robot description, xacro)
@@ -1,6 +1,5 @@
 <?xml version="1.0"?>
 <robot name="myrobotagv" xmlns:xacro="http://www.ros.org/wiki/xacro">
-    <xacro:include filename="$(find mobile_robot)/urdf/new_robot_2.xacro"/>
-    <xacro:include filename="$(find mobile_robot)/urdf/gazebo.xacro"/>
-    <xacro:include filename="$(find mobile_robot)/urdf/ros2_control.xacro"/>
+    <xacro:include filename="$(find amr_descriptions)/model/wheeled/urdf/mobile_robot.xacro"/>
+    <xacro:include filename="$(find amr_descriptions)/model/wheeled/urdf/gazebo.xacro"/>
 </robot>

File: src/amr_descriptions/model/wheeled/urdf/ros2_control.xacro (robot description, xacro)
@@ -25,5 +25,5 @@
     <gazebo>
         <plugin filename="gz_ros2_control-system" name="gz_ros2_control::GazeboSimROS2ControlPlugin">
-            <parameters>$(find mobile_robot)/config/my_controller.yaml</parameters>
+            <parameters>$(find amr_descriptions)/model/wheeled/config/ros2_control.yaml</parameters>
         </plugin>
         <plugin filename="ignition-gazebo-imu-system" name="ignition::gazebo::systems::Imu">

Commit message: feat: can control with keyboard

File: src/amr_descriptions/model/wheeled/urdf/gazebo.xacro (robot description, xacro)
@@ -7,7 +7,19 @@
     <gazebo reference="left_wheel">
         <material>Gazebo/Blue</material>
+        <mu1>1.0</mu1>
+        <mu2>1.0</mu2>
+        <kp>1000000.0</kp>
+        <kd>10.0</kd>
+        <minDepth>0.001</minDepth>
+        <maxVel>10.0</maxVel>
     </gazebo>
     <gazebo reference="right_wheel">
         <material>Gazebo/Blue</material>
+        <mu1>1.0</mu1>
+        <mu2>1.0</mu2>
+        <kp>1000000.0</kp>
+        <kd>10.0</kd>
+        <minDepth>0.001</minDepth>
+        <maxVel>10.0</maxVel>
     </gazebo>
         <gazebo reference="above_base_caster">

File: src/amr_descriptions/model/wheeled/urdf/mobile_robot.xacro (robot description, xacro)
@@ -36,21 +36,20 @@
 	</material>
 <!--define physical properties for robot-->
-	<xacro:property name="body_length" value="0.31"/>
+	<xacro:property name="robot_mass" value="4"/>
+	<xacro:property name="body_length" value="0.3"/>
 	<xacro:property name="body_width" value="0.4"/>
-	<xacro:property name="body_height" value="0.2"/>
-	<xacro:property name="body_mass" value="12"/>
-	<xacro:property name="base_caster_length" value="0.25"/>
-	<xacro:property name="base_caster_width" value="0.01"/>
-	<xacro:property name="base_caster_height" value="0.37"/>
-	<xacro:property name="above_base_caster_length" value="0.25"/>
-	<xacro:property name="above_base_caster_width" value="0.4"/>
-	<xacro:property name="above_base_caster_height" value="0.0075"/>
-	<xacro:property name="back_base_caster_length" value="0.0075"/>
-	<xacro:property name="back_base_caster_width" value="0.4"/>
-	<xacro:property name="back_base_caster_height" value="0.37"/>
+	<xacro:property name="body_height" value="0.3"/>
+	<xacro:property name="body_mass" value="15"/>
+	<!-- Frame structure properties (20x20cm grid) -->
+	<xacro:property name="frame_beam_radius" value="0.008"/>
+	<xacro:property name="frame_beam_mass" value="0.2"/>
+	<xacro:property name="frame_beam_20" value="0.02"/>
+	<xacro:property name="frame_beam_40" value="0.04"/>
+	<xacro:property name="mica_sheet_thickness" value="0.005"/>
+	<xacro:property name="mica_mass" value="0.2"/>
 	<xacro:property name="wheel_radius" value="0.05"/>
 	<xacro:property name="wheel_width" value="0.03"/>
 	<xacro:property name="wheel_mass" value="0.3"/>
-	<xacro:property name="wheel_separation" value="0.46"/>
+	<xacro:property name="wheel_separation" value="0.42"/>
 	<xacro:property name="PI" value="3.1415926535897931"/>
 	<xacro:macro name="cylinder_inertia" params="m r h">
@@ -75,29 +74,193 @@
 	<link name="base_link">
        	<origin xyz="0.0 0.0 0.0"/>
-    </link>
-<!--chassis link-->
+       	<inertial>
+       		<origin xyz="0.0 0.0 0.0" rpy="0.0 0.0 0.0"/>
+       		<mass value="${robot_mass}"/>
+       		<inertia ixx="0.5" ixy="0.0" ixz="0.0" iyy="0.5" iyz="0.0" izz="0.5"/>
+       	</inertial>
+    </link>
+<!--chassis link - Frame Structure with Grid-->
     <joint name="chassis_joint" type="fixed">
         <parent link="base_link"/>
         <child link="chassis"/>
-        <origin xyz="0.16 0.0 0.0"/>
+        <origin xyz="0.0 0.0 0.0"/>
     </joint>
     <link name="chassis">
         <visual>
-            <origin xyz="-0.2055 0.0 0.07" rpy="0.0 0.0 0.0"/>
-            <geometry>
-                 <box size="${body_length} ${body_width} ${body_height}"/>
-            </geometry>
-            <material name="yellow"/>
-        </visual>
-        <collision>
-            <origin xyz="-0.2055 0.0 0.07" rpy="0.0 0.0 0.0"/>
-            <geometry>
-                 <box size="${body_length} ${body_width} ${body_height}"/>
-            </geometry>
-        </collision>
-        <inertial>
-            <origin xyz="-0.2055 0.0 0.07" rpy="0.0 0.0 0.0"/>
-            <mass value="${body_mass}"/>
-            <xacro:box_inertia m="${body_mass}" l="${body_length}" w="${body_width}" h="${body_height}"/>
+            <origin xyz="0.0 0.0 0.0" rpy="0.0 0.0 0.0"/>
+            <geometry>
+                 <box size="${body_length} ${body_width} ${mica_sheet_thickness}"/>
+            </geometry>
+            <material name="white"/>
+        </visual>
+        <collision>
+            <origin xyz="0.0 0.0 0.0" rpy="0.0 0.0 0.0"/>
+            <geometry>
+                 <box size="${body_length} ${body_width} ${mica_sheet_thickness}"/>
+            </geometry>
+        </collision>
+        <inertial>
+            <origin xyz="0.0 0.0 0.0" rpy="0.0 0.0 0.0"/>
+            <mass value="${mica_mass}"/>
+            <xacro:box_inertia m="${mica_mass}" l="${body_length}" w="${body_width}" h="${mica_sheet_thickness}"/>
+        </inertial>
+    </link>
+    <!-- Vertical support posts (corners) -->
+    <!-- Front Left Post -->
+    <joint name="post_fl_joint" type="fixed">
+        <parent link="base_link"/>
+        <child link="post_fl"/>
+        <origin xyz="0.15 -0.2 0.15"/>
+    </joint>
+    <link name="post_fl">
+        <visual>
+            <origin xyz="0.0 0.0 0.0" rpy="0.0 0.0 0.0"/>
+            <geometry>
+                <box size="${frame_beam_20} ${frame_beam_20} ${body_height}"/>
+            </geometry>
+            <material name="aluminium"/>
+        </visual>
+        <collision>
+            <origin xyz="0.0 0.0 0.0" rpy="0.0 0.0 0.0"/>
+            <geometry>
+                <box size="${frame_beam_20} ${frame_beam_20} ${body_height}"/>
+            </geometry>
+        </collision>
+        <inertial>
+            <origin xyz="0.0 0.0 0.0" rpy="0.0 0.0 0.0"/>
+            <mass value="${frame_beam_mass}"/>
+            <xacro:box_inertia m="${frame_beam_mass}" l="${frame_beam_20}" w="${frame_beam_20}" h="${body_height}"/>
+        </inertial>
+    </link>
+    <!-- Front Right Post -->
+    <joint name="post_fr_joint" type="fixed">
+        <parent link="base_link"/>
+        <child link="post_fr"/>
+        <origin xyz="0.15 0.2 0.15"/>
+    </joint>
+    <link name="post_fr">
+        <visual>
+            <origin xyz="0.0 0.0 0.0" rpy="0.0 0.0 0.0"/>
+            <geometry>
+                <box size="${frame_beam_20} ${frame_beam_20} ${body_height}"/>
+            </geometry>
+            <material name="aluminium"/>
+        </visual>
+        <collision>
+            <origin xyz="0.0 0.0 0.0" rpy="0.0 0.0 0.0"/>
+            <geometry>
+                <box size="${frame_beam_20} ${frame_beam_20} ${body_height}"/>
+            </geometry>
+        </collision>
+        <inertial>
+            <origin xyz="0.0 0.0 0.0" rpy="0.0 0.0 0.0"/>
+            <mass value="${frame_beam_mass}"/>
+            <xacro:box_inertia m="${frame_beam_mass}" l="${frame_beam_20}" w="${frame_beam_20}" h="${body_height}"/>
+        </inertial>
+    </link>
+    <!-- Back Left Post -->
+    <joint name="post_bl_joint" type="fixed">
+        <parent link="base_link"/>
+        <child link="post_bl"/>
+        <origin xyz="-0.15 -0.2 0.15"/>
+    </joint>
+    <link name="post_bl">
+        <visual>
+            <origin xyz="0.0 0.0 0.0" rpy="0.0 0.0 0.0"/>
+            <geometry>
+                <box size="${frame_beam_20} ${frame_beam_20} ${body_height}"/>
+            </geometry>
+            <material name="aluminium"/>
+        </visual>
+        <collision>
+            <origin xyz="0.0 0.0 0.0" rpy="0.0 0.0 0.0"/>
+            <geometry>
+                <box size="${frame_beam_20} ${frame_beam_20} ${body_height}"/>
+            </geometry>
+        </collision>
+        <inertial>
+            <origin xyz="0.0 0.0 0.0" rpy="0.0 0.0 0.0"/>
+            <mass value="${frame_beam_mass}"/>
+            <xacro:box_inertia m="${frame_beam_mass}" l="${frame_beam_20}" w="${frame_beam_20}" h="${body_height}"/>
+        </inertial>
+    </link>
+    <!-- Back Right Post -->
+    <joint name="post_br_joint" type="fixed">
+        <parent link="base_link"/>
+        <child link="post_br"/>
+        <origin xyz="-0.15 0.2 0.15"/>
+    </joint>
+    <link name="post_br">
+        <visual>
+            <origin xyz="0.0 0.0 0.0" rpy="0.0 0.0 0.0"/>
+            <geometry>
+                <box size="${frame_beam_20} ${frame_beam_20} ${body_height}"/>
+            </geometry>
+            <material name="aluminium"/>
+        </visual>
+        <collision>
+            <origin xyz="0.0 0.0 0.0" rpy="0.0 0.0 0.0"/>
+            <geometry>
+                <box size="${frame_beam_20} ${frame_beam_20} ${body_height}"/>
+            </geometry>
+        </collision>
+        <inertial>
+            <origin xyz="0.0 0.0 0.0" rpy="0.0 0.0 0.0"/>
+            <mass value="${frame_beam_mass}"/>
+            <xacro:box_inertia m="${frame_beam_mass}" l="${frame_beam_20}" w="${frame_beam_20}" h="${body_height}"/>
+        </inertial>
+    </link>
+    <!-- Middle vertical posts (20x20cm grid) -->
+    <!-- Mica layers at different heights -->
+    <!-- Middle Layer -->
+    <joint name="layer_middle_joint" type="fixed">
+        <parent link="base_link"/>
+        <child link="layer_middle"/>
+        <origin xyz="0.0 0.0 0.15" rpy="0.0 0.0 0.0"/>
+    </joint>
+    <link name="layer_middle">
+        <visual>
+            <origin xyz="0.0 0.0 0.0" rpy="0.0 0.0 0.0"/>
+            <geometry>
+                 <box size="${body_length} ${body_width} ${mica_sheet_thickness}"/>
+            </geometry>
+            <material name="white"/>
+        </visual>
+        <collision>
+            <origin xyz="0.0 0.0 0.0" rpy="0.0 0.0 0.0"/>
+            <geometry>
+                 <box size="${body_length} ${body_width} ${mica_sheet_thickness}"/>
+            </geometry>
+        </collision>
+        <inertial>
+            <origin xyz="0.0 0.0 0.0" rpy="0.0 0.0 0.0"/>
+            <mass value="${mica_mass}"/>
+            <xacro:box_inertia m="${mica_mass}" l="${body_length}" w="${body_width}" h="${mica_sheet_thickness}"/>
+        </inertial>
+    </link>
+    <!-- Top Layer -->
+    <joint name="layer_top_joint" type="fixed">
+        <parent link="base_link"/>
+        <child link="layer_top"/>
+        <origin xyz="0.0 0.0 0.295" rpy="0.0 0.0 0.0"/>
+    </joint>
+    <link name="layer_top">
+        <visual>
+            <origin xyz="0.0 0.0 0.0" rpy="0.0 0.0 0.0"/>
+            <geometry>
+                 <box size="${body_length} ${body_width} ${mica_sheet_thickness}"/>
+            </geometry>
+            <material name="white"/>
+        </visual>
+        <collision>
+            <origin xyz="0.0 0.0 0.0" rpy="0.0 0.0 0.0"/>
+            <geometry>
+                 <box size="${body_length} ${body_width} ${mica_sheet_thickness}"/>
+            </geometry>
+        </collision>
+        <inertial>
+            <origin xyz="0.0 0.0 0.0" rpy="0.0 0.0 0.0"/>
+            <mass value="${mica_mass}"/>
+            <xacro:box_inertia m="${mica_mass}" l="${body_length}" w="${body_width}" h="${mica_sheet_thickness}"/>
         </inertial>
     </link>
@@ -106,5 +269,5 @@
         <parent link="base_link"/>
         <child link="right_wheel"/>
-        <origin xyz="0.03 -0.23 0.0" rpy="${PI/2} 0 0"/>
+        <origin xyz="0.1 -0.23 0.0" rpy="${PI/2} 0 0"/>
         <axis xyz="0 0 -1"/>
     </joint>
@@ -130,5 +293,5 @@
        	<parent link="base_link"/>
         <child link="left_wheel"/>
-        <origin xyz="0.03 0.23 0.0" rpy="${-PI/2} 0.0 0.0"/>
+        <origin xyz="0.1 0.23 0.0" rpy="${-PI/2} 0.0 0.0"/>
         <axis xyz="0 0 1"/>
     </joint>
@@ -150,139 +313,36 @@
         </inertial>
 	</link>
-<!--base caster-->
-	<!--above-->
-	<joint name="above_base_caster_joint" type="fixed">
-         	<parent link="base_link"/>
-         	<child link="above_base_caster"/>
-         	<origin xyz="-0.025 0.0 0.40" rpy="0 0 0"/>
-    </joint>
-	<link name = "above_base_caster" >
+<!--caster wheel - free castor at back-->
+	<joint name="caster_wheel_joint" type="fixed">
+		<parent link="base_link"/>
+		<child link="caster_wheel"/>
+		<origin xyz="-0.1 0.0 -0.035"/>
+	</joint>
+	<link name="caster_wheel">
 		<visual>
 			<geometry>
-				<box size="${above_base_caster_length} ${above_base_caster_width} ${above_base_caster_height}"/>
+				<sphere radius="0.035"/>
 			</geometry>
-			<material name = "orange" />
+			<material name="red"/>
 		</visual>
 		<collision>
 			<geometry>
-				<box size="${above_base_caster_length} ${above_base_caster_width} ${above_base_caster_height}"/>
+				<sphere radius="0.035"/>
 			</geometry>
 		</collision>
 		<inertial>
-            <mass value="0.2" />
-            <inertia ixx="0.1" ixy="0.0" ixz="0.0"
-                iyy="0.1" iyz="0.0"
-                izz="0.1" />
-        	</inertial>
-	</link>
-	<!--right-->
-	<joint name="right_base_caster_joint" type="fixed">
-        <parent link="base_link"/>
-        <child link="right_base_caster"/>
-        <origin xyz="-0.025 0.19 0.22" rpy="0 0 0"/>
-    </joint>
-	<link name = "right_base_caster" >
-		<visual>
-			<geometry>
-				<box size="${base_caster_length} ${base_caster_width} ${base_caster_height}"/>
-			</geometry>
-			<material name = "orange" />
-		</visual>
-		<collision>
-			<geometry>
-				<box size="${base_caster_length} ${base_caster_width} ${base_caster_height}"/>
-			</geometry>
-		</collision>
-		<inertial>
-        	<mass value="0.2" />
-            <inertia ixx="0.1" ixy="0.0" ixz="0.0"
-                iyy="0.1" iyz="0.0"
-                izz="0.1" />
-        	</inertial>
-	</link>
-	<!--left-->
-	<joint name="left_base_caster_joint" type="fixed">
-        <parent link="base_link"/>
-        <child link="left_base_caster"/>
-        <origin xyz="-0.025 -0.19 0.22" rpy="0 0 0"/>
-    </joint>
-	<link name = "left_base_caster" >
-		<visual>
-			<geometry>
-				<box size="${base_caster_length} ${base_caster_width} ${base_caster_height}"/>
-			</geometry>
-			<material name = "orange" />
-		</visual>
-		<collision>
-			<geometry>
-				<box size="${base_caster_length} ${base_caster_width} ${base_caster_height}"/>
-			</geometry>
-		</collision>
-		<inertial>
-            <mass value="0.2" />
-            <inertia ixx="0.1" ixy="0.0" ixz="0.0"
-                iyy="0.1" iyz="0.0"
-                izz="0.1" />
-        </inertial>
-	</link>
-	<!--back-->
-	<joint name="back_base_caster_joint" type="fixed">
-        <parent link="base_link"/>
-        <child link="back_base_caster"/>
-        <origin xyz="0.1 0 0.22" rpy="0 0 0"/>
-    </joint>
-	<link name = "back_base_caster" >
-		<visual>
-			<geometry>
-				<box size="${back_base_caster_length} ${back_base_caster_width} ${back_base_caster_height}"/>
-			</geometry>
-			<material name = "orange" />
-		</visual>
-		<collision>
-			<geometry>
-				<box size="${base_caster_length} ${base_caster_width} ${base_caster_height}"/>
-			</geometry>
-		</collision>
-		<inertial>
-            <mass value="0.5" />
-            <inertia ixx="0.1" ixy="0.0" ixz="0.0"
-            	iyy="0.1" iyz="0.0"
-                izz="0.1" />
-        	</inertial>
-	</link>
-<!--caster wheel-->
-	<joint name = "caster_wheel_joint" type = "fixed" >
-		<parent link = "base_link" />
-		<child link = "caster_wheel" />
-		<origin xyz = "-0.13 0 0.0" />
-	</joint>
-	<link name = "caster_wheel" >
-		<visual>
-			<geometry>
-				<sphere radius = "0.05" />
-			</geometry>
-			<material name = "red" />
-		</visual>
-		<collision>
-			<geometry>
-				<sphere radius = "0.05" />
-			</geometry>
-		</collision>
-		<inertial>
-            <mass value="0.1" />
-            <inertia ixx="0.1" ixy="0.0" ixz="0.0"
-                iyy="0.1" iyz="0.0"
-                izz="0.1" />
-        </inertial>
+			<mass value="0.08"/>
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