Commit message: feat: can localization with gazebo and mapping

File: src/amr_descriptions/model/wheeled/urdf/gazebo.xacro (robot description, xacro)
@@ -1,6 +1,5 @@
 <?xml version="1.0" ?>
 <robot name="diff_drive" xmlns:xacro="http://ros.org/wiki/xacro">
-<!--define robot gazebo-->
-        <gazebo reference="chassis">
+    <gazebo reference="chassis">
         <material>Gazebo/Aluminium</material>
     </gazebo>
@@ -23,5 +22,5 @@
         <maxVel>10.0</maxVel>
     </gazebo>
-        <gazebo reference="above_base_caster">
+    <gazebo reference="above_base_caster">
         <material>Gazebo/Yellow</material>
     </gazebo>
@@ -29,29 +28,25 @@
         <material>Gazebo/Yellow</material>
     </gazebo>
-        <gazebo reference="left_base_caster">
+    <gazebo reference="left_base_caster">
         <material>Gazebo/Yellow</material>
     </gazebo>
-        <gazebo reference="back_base_caster">
+    <gazebo reference="back_base_caster">
         <material>Gazebo/Yellow</material>
     </gazebo>
-        <gazebo reference="caster_wheel">
+    <gazebo reference="caster_wheel">
+        <material>Gazebo/Red</material>
+        <mu1>0.0</mu1>
+        <mu2>0.0</mu2>
+        <kp>1000000.0</kp>
+        <kd>100.0</kd>
+        <minDepth>0.001</minDepth>
+        <maxVel>1.0</maxVel>
+    </gazebo>
+    <gazebo reference="face_link">
         <material>Gazebo/Red</material>
     </gazebo>
-        <gazebo reference="face_link">
-        <material>Gazebo/Red</material>
-    </gazebo>
-        <gazebo reference="laser">
+    <gazebo reference="laser">
         <material>Gazebo/Orange</material>
     </gazebo>
-  <!-- Caster wheel -->
-  <gazebo reference="caster_wheel">
-    <mu1>0.0</mu1>
-    <mu2>0.0</mu2>
-    <kp>1000000.0</kp>
-    <kd>100.0</kd>
-    <minDepth>0.001</minDepth>
-    <maxVel>1.0</maxVel>
-  </gazebo>
-    <!-- LIDAR sensor cho Gazebo Fortress -->
     <gazebo reference="laser">
         <sensor name="laser" type="gpu_ray">
@@ -83,160 +78,91 @@
         </sensor>
     </gazebo>
-    <!-- IMU -->
-  <gazebo reference="imu_link">
-    <sensor name="imu" type="imu">
-        <always_on>true</always_on>
-        <update_rate>100</update_rate>
-        <gz_frame_id>imu_link</gz_frame_id>
-        <topic>imu</topic>
-        <imu>
-          <angular_velocity>
-            <x>
-              <noise type="gaussian">
-                <mean>0.0</mean>
-                <stddev>2e-4</stddev>
-              </noise>
-            </x>
-            <y>
-              <noise type="gaussian">
-                <mean>0.0</mean>
-                <stddev>2e-4</stddev>
-              </noise>
-            </y>
-            <z>
-              <noise type="gaussian">
-                <mean>0.0</mean>
-                <stddev>2e-4</stddev>
-              </noise>
-            </z>
-          </angular_velocity>
-          <linear_acceleration>
-            <x>
-              <noise type="gaussian">
-                <mean>0.0</mean>
-                <stddev>1.7e-2</stddev>
-              </noise>
-            </x>
-            <y>
-              <noise type="gaussian">
-                <mean>0.0</mean>
-                <stddev>1.7e-2</stddev>
-              </noise>
-            </y>
-            <z>
-              <noise type="gaussian">
-                <mean>0.0</mean>
-                <stddev>1.7e-2</stddev>
-              </noise>
-            </z>
-          </linear_acceleration>
-        </imu>
-    </sensor>
-  </gazebo>
-  <!-- Depth Camera for Point Cloud (obstacle detection) -->
-  <gazebo reference="laser">
-    <sensor name="depth_camera" type="depth_camera">
-      <always_on>true</always_on>
-      <update_rate>30</update_rate>
-      <visualize>true</visualize>
-      <gz_frame_id>laser</gz_frame_id>
-      <topic>camera/points</topic>
-      <camera>
-        <horizontal_fov>1.57</horizontal_fov>
-        <vertical_fov>1.57</vertical_fov>
-        <image>
-          <width>640</width>
-          <height>480</height>
-          <format>R8G8B8</format>
-        </image>
-        <clip><near>0.1</near><far>10.0</far></clip>
-      </camera>
-      <noise><type>gaussian</type><mean>0.0</mean><stddev>0.01</stddev></noise>
-    </sensor>
-  </gazebo>
-  <!-- ZED2 Stereo Camera -->
-  <!-- Left camera -->
-<gazebo reference="zed2_left_camera_frame">
-  <sensor name="zed2_left_camera_sensor" type="camera">
-    <always_on>true</always_on>
-    <update_rate>30</update_rate>
-    <visualize>true</visualize>
-    <gz_frame_id>zed2_left_camera_frame</gz_frame_id>
-    <topic>zed2/left/image_raw</topic>
-    <camera_info_topic>zed2/left/camera_info</camera_info_topic>
-    <camera>
-      <horizontal_fov>1.92</horizontal_fov>
-      <vertical_fov>1.08</vertical_fov>
-      <image>
-        <width>1280</width>
-        <height>720</height>
-        <format>R8G8B8</format>
-      </image>
-      <clip><near>0.05</near><far>50.0</far></clip>
-    </camera>
-    <noise><type>gaussian</type><mean>0.0</mean><stddev>0.003</stddev></noise>
-  </sensor>
-</gazebo>
-<!-- Right camera -->
-<gazebo reference="zed2_right_camera_frame">
-  <sensor name="zed2_right_camera_sensor" type="camera">
-    <always_on>true</always_on>
-    <update_rate>30</update_rate>
-    <visualize>true</visualize>
-    <gz_frame_id>zed2_right_camera_frame</gz_frame_id>
-    <topic>zed2/right/image_raw</topic>
-    <camera_info_topic>zed2/right/camera_info</camera_info_topic>
-    <camera>
-      <horizontal_fov>1.92</horizontal_fov>
-      <vertical_fov>1.08</vertical_fov>
-      <image>
-        <width>1280</width>
-        <height>720</height>
-        <format>R8G8B8</format>
-      </image>
-      <clip><near>0.05</near><far>50.0</far></clip>
-    </camera>
-    <noise><type>gaussian</type><mean>0.0</mean><stddev>0.003</stddev></noise>
-  </sensor>
-</gazebo>
-  <!-- ============================================ -->
-  <!-- ROS2 CONTROL CONFIGURATION -->
-  <!-- ============================================ -->
-  <ros2_control name="GazeboSystem" type="system">
-    <hardware>
-      <plugin>gz_ros2_control/GazeboSimSystem</plugin>
-    </hardware>
-    <joint name="left_wheel_joint">
-      <command_interface name="velocity">
-        <param name="min">-10</param>
-        <param name="max">10</param>
-      </command_interface>
-      <state_interface name="velocity"/>
-      <state_interface name="position"/>
-    </joint>
-    <joint name="right_wheel_joint">
-      <command_interface name="velocity">
-        <param name="min">-10</param>
-        <param name="max">10</param>
-      </command_interface>
-      <state_interface name="velocity"/>
-      <state_interface name="position"/>
-    </joint>
-  </ros2_control>
-  <!-- ============================================ -->
-  <!-- GAZEBO PLUGINS -->
-  <!-- ============================================ -->
-  <gazebo>
-    <!-- ros2_control plugin -->
-    <plugin filename="libgz_ros2_control-system.so" name="gz_ros2_control::GazeboSimROS2ControlPlugin">
-      <parameters>$(find amr_descriptions)/model/wheeled/config/ros2_control.yaml</parameters>
-    </plugin>
-    <!-- IMU system -->
-    <plugin filename="gz-sim-imu-system" name="gz::sim::systems::Imu">
-    </plugin>
-    <!-- Sensors system for camera -->
-    <plugin filename="gz-sim-sensors-system" name="gz::sim::systems::Sensors">
-      <render_engine>ogre2</render_engine>
-    </plugin>
-  </gazebo>
+    <gazebo reference="imu_link">
+        <sensor name="imu" type="imu">
+            <always_on>true</always_on>
+            <update_rate>100</update_rate>
+            <gz_frame_id>imu_link</gz_frame_id>
+            <topic>imu</topic>
+            <imu>
+                <angular_velocity>
+                    <x><noise type="gaussian"><mean>0.0</mean><stddev>2e-4</stddev></noise></x>
+                    <y><noise type="gaussian"><mean>0.0</mean><stddev>2e-4</stddev></noise></y>
+                    <z><noise type="gaussian"><mean>0.0</mean><stddev>2e-4</stddev></noise></z>
+                </angular_velocity>
+                <linear_acceleration>
+                    <x><noise type="gaussian"><mean>0.0</mean><stddev>1.7e-2</stddev></noise></x>
+                    <y><noise type="gaussian"><mean>0.0</mean><stddev>1.7e-2</stddev></noise></y>
+                    <z><noise type="gaussian"><mean>0.0</mean><stddev>1.7e-2</stddev></noise></z>
+                </linear_acceleration>
+            </imu>
+        </sensor>
+    </gazebo>
+    <gazebo reference="zed2_left_camera_frame">
+        <sensor name="zed2_left_camera_sensor" type="rgbd_camera">
+            <always_on>true</always_on>
+            <update_rate>30</update_rate>
+            <visualize>true</visualize>
+            <gz_frame_id>zed2_left_camera_frame</gz_frame_id>
+            <topic>zed2/left</topic>
+            <camera>
+                <horizontal_fov>1.91986</horizontal_fov>
+                <image>
+                    <width>1280</width>
+                    <height>720</height>
+                    <format>R8G8B8</format>
+                </image>
+                <clip><near>0.2</near><far>20.0</far></clip>
+            </camera>
+            <noise><type>gaussian</type><mean>0.0</mean><stddev>0.003</stddev></noise>
+        </sensor>
+    </gazebo>
+    <gazebo reference="zed2_right_camera_frame">
+        <sensor name="zed2_right_camera_sensor" type="camera">
+            <always_on>true</always_on>
+            <update_rate>30</update_rate>
+            <visualize>false</visualize> <gz_frame_id>zed2_right_camera_frame</gz_frame_id>
+            <topic>zed2/right/image_raw</topic>
+            <camera_info_topic>zed2/right/camera_info</camera_info_topic>
+            <camera>
+                <horizontal_fov>1.91986</horizontal_fov>
+                <image>
+                    <width>1280</width>
+                    <height>720</height>
+                    <format>R8G8B8</format>
+                </image>
+                <clip><near>0.2</near><far>20.0</far></clip>
+            </camera>
+            <noise><type>gaussian</type><mean>0.0</mean><stddev>0.003</stddev></noise>
+        </sensor>
+    </gazebo>
+    <ros2_control name="GazeboSystem" type="system">
+        <hardware>
+            <plugin>gz_ros2_control/GazeboSimSystem</plugin>
+        </hardware>
+        <joint name="left_wheel_joint">
+            <command_interface name="velocity">
+                <param name="min">-10</param>
+                <param name="max">10</param>
+            </command_interface>
+            <state_interface name="velocity"/>
+            <state_interface name="position"/>
+        </joint>
+        <joint name="right_wheel_joint">
+            <command_interface name="velocity">
+                <param name="min">-10</param>
+                <param name="max">10</param>
+            </command_interface>
+            <state_interface name="velocity"/>
+            <state_interface name="position"/>
+        </joint>
+    </ros2_control>
+    <gazebo>
+        <plugin filename="libgz_ros2_control-system.so" name="gz_ros2_control::GazeboSimROS2ControlPlugin">
+            <parameters>$(find amr_descriptions)/model/wheeled/config/ros2_control.yaml</parameters>
+        </plugin>
+        <plugin filename="gz-sim-imu-system" name="gz::sim::systems::Imu"/>
+        <plugin filename="gz-sim-sensors-system" name="gz::sim::systems::Sensors">
+            <render_engine>ogre2</render_engine>
+        </plugin>
+    </gazebo>
 </robot>

File: src/amr_descriptions/model/wheeled/urdf/mobile_robot.xacro (robot description, xacro)
@@ -317,10 +317,10 @@
 		<parent link="base_link"/>
 		<child link="caster_wheel"/>
-		<origin xyz="-0.1 0.0 -0.035"/>
+		<origin xyz="-0.1 0.0 -0.015"/>
 	</joint>
 	<link name="caster_wheel">
 		<visual>
 			<geometry>
-				<sphere radius="0.035"/>
+				<sphere radius="0.015"/>
 			</geometry>
 			<material name="red"/>
