Commit message: feat: have update robot_description for realtime

File: src/descriptions/model/human/model.urdf (robot description, URDF)
Before this commit: robot human, 16 links, 15 joints
Links:
- removed link head
- removed link left_foot
- removed link left_forearm
- removed link left_hand
- removed link left_lower_leg
- removed link left_upper_arm
- removed link left_upper_leg
- removed link neck
- removed link pelvis
- removed link right_foot
- removed link right_forearm
- removed link right_hand
- removed link right_lower_leg
- removed link right_upper_arm
- removed link right_upper_leg
- removed link torso
- added link base_link, mass 65.0; collision cylinder length=1.8 radius=0.3; visual mesh filename=package://gazebo_ros/share/gazebo/models/walk_person/meshes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 scale=1 1 1
Joints:
- removed joint head_joint
- removed joint left_ankle_joint
- removed joint left_elbow_joint
- removed joint left_hip_joint
- removed joint left_knee_joint
- removed joint left_shoulder_joint
- removed joint left_wrist_joint
- removed joint neck_joint
- removed joint right_ankle_joint
- removed joint right_elbow_joint
- removed joint right_hip_joint
- removed joint right_knee_joint
- removed joint right_shoulder_joint
- removed joint right_wrist_joint
- removed joint torso_joint

File: src/descriptions/model/wheeled/urdf/gazebo.xacro (robot description, xacro)
@@ -78,10 +78,10 @@
         </sensor>
     </gazebo>
-    <gazebo reference="imu_link">
+    <gazebo reference="zed2_link">
         <sensor name="imu" type="imu">
             <always_on>true</always_on>
             <update_rate>100</update_rate>
-            <gz_frame_id>imu_link</gz_frame_id>
-            <topic>imu</topic>
+            <gz_frame_id>zed2_link</gz_frame_id>
+            <topic>/zed/zed_node/imu/data</topic>
             <imu>
                 <angular_velocity>
@@ -104,5 +104,5 @@
             <visualize>true</visualize>
             <gz_frame_id>zed2_left_camera_frame</gz_frame_id>
-            <topic>zed2/left</topic>
+            <topic>/zed/zed_node/left/image_rect_color</topic>
             <camera>
                 <horizontal_fov>1.91986</horizontal_fov>
@@ -140,4 +140,35 @@
             <plugin>gz_ros2_control/GazeboSimSystem</plugin>
         </hardware>
+    <gazebo reference="zed2_right_camera_frame">
+        <sensor name="zed2_right_camera_sensor" type="camera">
+            <always_on>true</always_on>
+            <update_rate>30</update_rate>
+            <visualize>false</visualize> <gz_frame_id>zed2_right_camera_frame</gz_frame_id>
+            <topic>zed2/right/image_raw</topic>
+            <camera_info_topic>zed2/right/camera_info</camera_info_topic>
+            <camera>
+                <horizontal_fov>1.91986</horizontal_fov>
+                <image>
+                    <width>1280</width>
+                    <height>720</height>
+                    <format>R8G8B8</format>
+                </image>
+                <clip><near>0.2</near><far>20.0</far></clip>
+            </camera>
+            <noise><type>gaussian</type><mean>0.0</mean><stddev>0.003</stddev></noise>
+        </sensor>
+    </gazebo>
+    <ros2_control name="GazeboSystem" type="system">
+        <hardware>
+            <plugin>gz_ros2_control/GazeboSimSystem</plugin>
+        </hardware>
+        <joint name="left_wheel_joint">
+            <command_interface name="velocity">
+                <param name="min">-10</param>
+                <param name="max">10</param>
+            </command_interface>
+            <state_interface name="velocity"/>
+            <state_interface name="position"/>
+        </joint>
         <joint name="left_wheel_joint">
             <command_interface name="velocity">
@@ -166,3 +197,21 @@
         </plugin>
     </gazebo>
+        <joint name="right_wheel_joint">
+            <command_interface name="velocity">
+                <param name="min">-10</param>
+                <param name="max">10</param>
+            </command_interface>
+            <state_interface name="velocity"/>
+            <state_interface name="position"/>
+        </joint>
+    </ros2_control>
+    <gazebo>
+        <plugin filename="libgz_ros2_control-system.so" name="gz_ros2_control::GazeboSimROS2ControlPlugin">
+            <parameters>$(find descriptions)/model/wheeled/config/ros2_control.yaml</parameters>
+        </plugin>
+        <plugin filename="gz-sim-imu-system" name="gz::sim::systems::Imu"/>
+        <plugin filename="gz-sim-sensors-system" name="gz::sim::systems::Sensors">
+            <render_engine>ogre2</render_engine>
+        </plugin>
+    </gazebo>
 </robot>

File: src/descriptions/model/wheeled/urdf/mobile_robot.xacro (robot description, xacro)
@@ -1,7 +1,5 @@
 <?xml version="1.0"?>
 <robot xmlns:xacro="http://www.ros.org/wiki/xacro">
-    <xacro:include filename="$(find descriptions)/model/wheeled/urdf/zed_macro.urdf.xacro"/>
-<!--matierials.xacro-->
-	<material name="black">
+<material name="black">
 		<color rgba="0.0 0.0 0.0 1.0"/>
 	</material>
@@ -36,11 +34,9 @@
 		<color rgba="${132/255} ${135/255} ${137/255} 1.0"/>
 	</material>
-<!--define physical properties for robot-->
-	<xacro:property name="robot_mass" value="4"/>
+<xacro:property name="robot_mass" value="4"/>
 	<xacro:property name="body_length" value="0.3"/>
 	<xacro:property name="body_width" value="0.4"/>
 	<xacro:property name="body_height" value="0.3"/>
 	<xacro:property name="body_mass" value="15"/>
-	<!-- Frame structure properties (20x20cm grid) -->
 	<xacro:property name="frame_beam_radius" value="0.008"/>
 	<xacro:property name="frame_beam_mass" value="0.2"/>
@@ -64,7 +60,6 @@
 		         izz="${m*(w*w+l*l)/12}" />
 	</xacro:macro>
-<!--base link-->
-    <joint name="base_footprint_joint" type="fixed">
-       	<origin xyz="0.0 0.0 ${wheel_radius}" rpy="0.0 0.0 0.0"/>
+<joint name="base_footprint_joint" type="fixed">
+    	<origin xyz="0.0 0.0 ${wheel_radius}" rpy="0.0 0.0 0.0"/>
         <parent link="base_footprint"/>
         <child link="base_link"/>
@@ -81,6 +76,5 @@
        	</inertial>
     </link>
-<!--chassis link - Frame Structure with Grid-->
-    <joint name="chassis_joint" type="fixed">
+<joint name="chassis_joint" type="fixed">
         <parent link="base_link"/>
         <child link="chassis"/>
@@ -107,6 +101,4 @@
         </inertial>
     </link>
-    <!-- Vertical support posts (corners) -->
-    <!-- Front Left Post -->
     <joint name="post_fl_joint" type="fixed">
         <parent link="base_link"/>
@@ -134,5 +126,4 @@
         </inertial>
     </link>
-    <!-- Front Right Post -->
     <joint name="post_fr_joint" type="fixed">
         <parent link="base_link"/>
@@ -160,5 +151,4 @@
         </inertial>
     </link>
-    <!-- Back Left Post -->
     <joint name="post_bl_joint" type="fixed">
         <parent link="base_link"/>
@@ -186,5 +176,4 @@
         </inertial>
     </link>
-    <!-- Back Right Post -->
     <joint name="post_br_joint" type="fixed">
         <parent link="base_link"/>
@@ -212,7 +201,4 @@
         </inertial>
     </link>
-    <!-- Middle vertical posts (20x20cm grid) -->
-    <!-- Mica layers at different heights -->
-    <!-- Middle Layer -->
     <joint name="layer_middle_joint" type="fixed">
         <parent link="base_link"/>
@@ -240,5 +226,4 @@
         </inertial>
     </link>
-    <!-- Top Layer -->
     <joint name="layer_top_joint" type="fixed">
         <parent link="base_link"/>
@@ -266,6 +251,5 @@
         </inertial>
     </link>
-<!--right wheel-->
-    <joint name="right_wheel_joint" type="continuous">
+<joint name="right_wheel_joint" type="continuous">
         <parent link="base_link"/>
         <child link="right_wheel"/>
@@ -290,6 +274,5 @@
         	</inertial>
     </link>
-<!--left wheel-->
-	<joint name="left_wheel_joint" type="continuous">
+<joint name="left_wheel_joint" type="continuous">
        	<parent link="base_link"/>
         <child link="left_wheel"/>
@@ -314,6 +297,5 @@
         </inertial>
 	</link>
-<!--caster wheel - free castor at back-->
-	<joint name="caster_wheel_joint" type="fixed">
+<joint name="caster_wheel_joint" type="fixed">
 		<parent link="base_link"/>
 		<child link="caster_wheel"/>
@@ -329,5 +311,5 @@
 		<collision>
 			<geometry>
-				<sphere radius="0.035"/>
+				<sphere radius="0.015"/>
 			</geometry>
 		</collision>
@@ -337,6 +319,5 @@
 		</inertial>
 	</link>
-<!--lidar-->
-	<joint name="joint_scan" type="fixed">
+<joint name="joint_scan" type="fixed">
 		<origin xyz="0.0 0.0 0.4" rpy="0 0 0"/>
 		<parent link="base_link"/>
@@ -357,21 +338,40 @@
         </inertial>
     </link>
-    <!-- Manufacturer ZED2 macro instance -->
-    <joint name="zed2_mount_joint" type="fixed">
-        <parent link="base_link"/>
-        <child link="zed2_camera_link"/>
-        <origin xyz="0.15 0.0 0.35" rpy="0 0 0"/>
-    </joint>
-    <xacro:zed_camera name="zed2" model="zed2">
-        <origin xyz="0 0 0" rpy="0 0 0"/>
-    </xacro:zed_camera>
-    <!-- Custom ZED2 geometry removed: using vendor zed_macro to avoid duplicated frames. -->
-	<!-- IMU (trên mặt robot, chính giữa thân) -->
-    <link name="imu_link"/>
-    <joint name="imu_joint" type="fixed">
-        <parent link="base_link"/>
-        <child link="imu_link"/>
-        <origin xyz="0.0 0.0 0.35" rpy="0 0 0"/>
-    </joint>
-    <!-- End IMU -->
-</robot>
+	<link name="zed2_camera_link">
+		<visual>
+			<origin xyz="0 0 0" rpy="0 0 0"/>
+			<geometry>
+				<box size="0.03 0.1465 0.023"/>
+			</geometry>
+			<material name="grey"/>
+		</visual>
+		<collision>
+			<origin xyz="0 0 0" rpy="0 0 0"/>
+			<geometry>
+				<box size="0.03 0.1465 0.023"/>
+			</geometry>
+		</collision>
+		<inertial>
+			<mass value="0.5"/>
+			<origin xyz="0 0 0" rpy="0 0 0"/>
+			<inertia ixx="0.01" iyy="0.01" izz="0.01" ixy="0" ixz="0" iyz="0"/>
+		</inertial>
+	</link>
+	<joint name="zed2_joint" type="fixed">
+		<parent link="base_link"/>
+		<child link="zed2_camera_link"/>
+		<origin xyz="0.15 0.0 0.35"/>
+	</joint>
+	<link name="zed2_left_camera_frame"/>
+	<joint name="zed2_left_camera_joint" type="fixed">
+		<parent link="zed2_camera_link"/>
+		<child link="zed2_left_camera_frame"/>
+		<origin xyz="0 -0.07325 0"/>
+	</joint>
+	<link name="zed2_right_camera_frame"/>
+	<joint name="zed2_right_camera_joint" type="fixed">
+		<parent link="zed2_camera_link"/>
+		<child link="zed2_right_camera_frame"/>
+		<origin xyz="0 0.07325 0"/>
+	</joint>
+	</robot>
