Commit message: feat: can initilizate robot_descripstion

File: src/descriptions/model/wheeled/urdf/mobile_robot.urdf.xacro (robot description, xacro)
@@ -1,5 +1,9 @@
 <?xml version="1.0"?>
-<robot name="myrobotagv" xmlns:xacro="http://www.ros.org/wiki/xacro">
-    <xacro:include filename="$(find descriptions)/model/wheeled/urdf/mobile_robot.xacro"/>
-    <xacro:include filename="$(find descriptions)/model/wheeled/urdf/gazebo.xacro"/>
+<robot xmlns:xacro="http://www.ros.org/wiki/xacro" name="mobile_robot">
+    <xacro:arg name="is_sim" default="false"/>
+    <xacro:include filename="mobile_robot.xacro" />
+    <xacro:include filename="ros2_control.xacro" />
+    <xacro:if value="$(arg is_sim)">
+        <xacro:include filename="gazebo.xacro" />
+    </xacro:if>
 </robot>

File: src/descriptions/model/wheeled/urdf/mobile_robot.xacro (robot description, xacro)
@@ -338,5 +338,5 @@
         </inertial>
     </link>
-	<link name="zed2_camera_link">
+	<link name="zed_camera_link">
 		<visual>
 			<origin xyz="0 0 0" rpy="0 0 0"/>
@@ -360,10 +360,10 @@
 	<joint name="zed2_joint" type="fixed">
 		<parent link="base_link"/>
-		<child link="zed2_camera_link"/>
+		<child link="zed_camera_link"/>
 		<origin xyz="0.15 0.0 0.35"/>
 	</joint>
 	<link name="zed2_left_camera_frame"/>
 	<joint name="zed2_left_camera_joint" type="fixed">
-		<parent link="zed2_camera_link"/>
+		<parent link="zed_camera_link"/>
 		<child link="zed2_left_camera_frame"/>
 		<origin xyz="0 -0.07325 0"/>
@@ -371,5 +371,5 @@
 	<link name="zed2_right_camera_frame"/>
 	<joint name="zed2_right_camera_joint" type="fixed">
-		<parent link="zed2_camera_link"/>
+		<parent link="zed_camera_link"/>
 		<child link="zed2_right_camera_frame"/>
 		<origin xyz="0 0.07325 0"/>

File: src/hardware_interfaces/zed2/zed_wrapper/urdf/zed_descr.urdf.xacro (robot description, xacro)
@@ -16,6 +16,6 @@
 -->
 <robot name="stereolabs_camera" xmlns:xacro="http://ros.org/wiki/xacro">
-  <xacro:arg name="camera_name"   default="zed" />
-  <xacro:arg name="camera_model"  default="zed" />
+  <xacro:arg name="camera_name"   default="zed2" />
+  <xacro:arg name="camera_model"  default="zed2" />
   <xacro:arg name="custom_baseline"  default="0.0" />
   <!-- If GNSS fusion is enabled the position of the antenna with respect to the camera mount point is required -->
