Commit message: feat: can simu stable on gazebo with RL

File: src/descriptions/model/wheeled/urdf/mobile_robot.xacro (robot description, xacro)
@@ -48,5 +48,5 @@
 	<xacro:property name="wheel_width" value="0.03"/>
 	<xacro:property name="wheel_mass" value="0.3"/>
-	<xacro:property name="wheel_separation" value="0.42"/>
+	<xacro:property name="wheel_separation" value="0.5"/>
 	<xacro:property name="PI" value="3.1415926535897931"/>
 	<xacro:macro name="cylinder_inertia" params="m r h">
@@ -300,10 +300,10 @@
 		<parent link="base_link"/>
 		<child link="caster_wheel"/>
-		<origin xyz="-0.1 0.0 -0.015"/>
+		<origin xyz="-0.1 0.0 -0.022"/>
 	</joint>
 	<link name="caster_wheel">
 		<visual>
 			<geometry>
-				<sphere radius="0.015"/>
+				<sphere radius="0.03"/>
 			</geometry>
 			<material name="red"/>
@@ -311,5 +311,5 @@
 		<collision>
 			<geometry>
-				<sphere radius="0.015"/>
+				<sphere radius="0.03"/>
 			</geometry>
 		</collision>

Commit message: feat: stay when initial Mapping on Rviz2

File: src/descriptions/model/wheeled/urdf/mobile_robot.xacro (robot description, xacro)
@@ -320,5 +320,5 @@
 	</link>
 <joint name="joint_scan" type="fixed">
-		<origin xyz="0.0 0.0 0.4" rpy="0 0 0"/>
+		<origin xyz="0.0 0.0 0.4" rpy="0 0 ${PI}"/>
 		<parent link="base_link"/>
 		<child link="laser"/>

Commit message: feat

File: src/descriptions/model/wheeled/urdf/mobile_robot.xacro (robot description, xacro)
@@ -338,5 +338,5 @@
         </inertial>
     </link>
-	<link name="zed_camera_link">
+	<link name="zed2_camera_link">
 		<visual>
 			<origin xyz="0 0 0" rpy="0 0 0"/>
@@ -360,5 +360,5 @@
 	<joint name="zed2_joint" type="fixed">
 		<parent link="base_link"/>
-		<child link="zed_camera_link"/>
+		<child link="zed2_camera_link"/>
 		<origin xyz="0.15 0.0 0.35"/>
 	</joint>
@@ -366,5 +366,5 @@
     <link name="zed2_link"/>
     <joint name="zed2_link_alias_joint" type="fixed">
-        <parent link="zed_camera_link"/>
+        <parent link="zed2_camera_link"/>
         <child link="zed2_link"/>
         <origin xyz="0 0 0" rpy="0 0 0"/>
@@ -372,5 +372,5 @@
 	<link name="zed2_left_camera_frame"/>
 	<joint name="zed2_left_camera_joint" type="fixed">
-		<parent link="zed_camera_link"/>
+		<parent link="zed2_camera_link"/>
 		<child link="zed2_left_camera_frame"/>
 		<origin xyz="0 -0.07325 0"/>
@@ -378,5 +378,5 @@
 	<link name="zed2_right_camera_frame"/>
 	<joint name="zed2_right_camera_joint" type="fixed">
-		<parent link="zed_camera_link"/>
+		<parent link="zed2_camera_link"/>
 		<child link="zed2_right_camera_frame"/>
 		<origin xyz="0 0.07325 0"/>

Commit message: feat: adjust zed2_link

File: src/descriptions/model/wheeled/urdf/mobile_robot.xacro (robot description, xacro)
@@ -338,47 +338,12 @@
         </inertial>
     </link>
-	<link name="zed2_camera_link">
-		<visual>
-			<origin xyz="0 0 0" rpy="0 0 0"/>
-			<geometry>
-				<box size="0.03 0.1465 0.023"/>
-			</geometry>
-			<material name="grey"/>
-		</visual>
-		<collision>
-			<origin xyz="0 0 0" rpy="0 0 0"/>
-			<geometry>
-				<box size="0.03 0.1465 0.023"/>
-			</geometry>
-		</collision>
-		<inertial>
-			<mass value="0.5"/>
-			<origin xyz="0 0 0" rpy="0 0 0"/>
-			<inertia ixx="0.01" iyy="0.01" izz="0.01" ixy="0" ixz="0" iyz="0"/>
-		</inertial>
-	</link>
-	<joint name="zed2_joint" type="fixed">
-		<parent link="base_link"/>
-		<child link="zed2_camera_link"/>
-		<origin xyz="0.15 0.0 0.35"/>
-	</joint>
-    <!-- Compatibility alias: keep legacy zed2_link frame for sensors/plugins -->
-    <link name="zed2_link"/>
-    <joint name="zed2_link_alias_joint" type="fixed">
-        <parent link="zed2_camera_link"/>
-        <child link="zed2_link"/>
+    <xacro:include filename="$(find zed_wrapper)/urdf/zed_macro.urdf.xacro" />
+    <xacro:zed_camera name="zed2" model="zed2" enable_gnss="false">
         <origin xyz="0 0 0" rpy="0 0 0"/>
-    </joint>
-	<link name="zed2_left_camera_frame"/>
-	<joint name="zed2_left_camera_joint" type="fixed">
-		<parent link="zed2_camera_link"/>
-		<child link="zed2_left_camera_frame"/>
-		<origin xyz="0 -0.07325 0"/>
-	</joint>
-	<link name="zed2_right_camera_frame"/>
-	<joint name="zed2_right_camera_joint" type="fixed">
-		<parent link="zed2_camera_link"/>
-		<child link="zed2_right_camera_frame"/>
-		<origin xyz="0 0.07325 0"/>
-	</joint>
-	</robot>
+    </xacro:zed_camera>
+    <joint name="zed2_base_joint" type="fixed">
+        <parent link="base_link"/>
+        <child link="zed2_camera_link"/>
+        <origin xyz="0.15 0.0 0.35" rpy="0 0 0"/>
+    </joint>
+</robot>

Commit message: feat: tuning ekf mapping, dont trust yaw of odom's zed2 when rotate

File: src/descriptions/model/wheeled/urdf/mobile_robot.xacro (robot description, xacro)
@@ -48,5 +48,5 @@
 	<xacro:property name="wheel_width" value="0.03"/>
 	<xacro:property name="wheel_mass" value="0.3"/>
-	<xacro:property name="wheel_separation" value="0.5"/>
+	<xacro:property name="wheel_separation" value="0.48"/>
 	<xacro:property name="PI" value="3.1415926535897931"/>
 	<xacro:macro name="cylinder_inertia" params="m r h">

Commit message: feat: yaw oke, linear not oke

File: src/descriptions/model/wheeled/urdf/mobile_robot.xacro (robot description, xacro)
@@ -35,7 +35,7 @@
 	</material>
 <xacro:property name="robot_mass" value="4"/>
-	<xacro:property name="body_length" value="0.3"/>
-	<xacro:property name="body_width" value="0.4"/>
-	<xacro:property name="body_height" value="0.3"/>
+	<xacro:property name="body_length" value="0.28"/>    <!-- 28cm dài (đổi từ 40cm) -->
+	<xacro:property name="body_width" value="0.4"/>     <!-- 40cm rộng (đổi từ 28cm) -->
+	<xacro:property name="body_height" value="0.4"/>    <!-- 40cm cao -->
 	<xacro:property name="body_mass" value="15"/>
 	<xacro:property name="frame_beam_radius" value="0.008"/>
@@ -43,10 +43,10 @@
 	<xacro:property name="frame_beam_20" value="0.02"/>
 	<xacro:property name="frame_beam_40" value="0.04"/>
-	<xacro:property name="mica_sheet_thickness" value="0.005"/>
+	<xacro:property name="mica_sheet_thickness" value="0.005"/>   <!-- 0.5cm dày -->
 	<xacro:property name="mica_mass" value="0.2"/>
-	<xacro:property name="wheel_radius" value="0.05"/>
+	<xacro:property name="wheel_radius" value="0.05"/>  <!-- 10cm đường kính, tức 5cm radius -->
 	<xacro:property name="wheel_width" value="0.03"/>
 	<xacro:property name="wheel_mass" value="0.3"/>
-	<xacro:property name="wheel_separation" value="0.48"/>
+	<xacro:property name="wheel_separation" value="0.46"/>  <!-- 46cm khoảng cách 2 bánh -->
 	<xacro:property name="PI" value="3.1415926535897931"/>
 	<xacro:macro name="cylinder_inertia" params="m r h">
@@ -61,5 +61,5 @@
 	</xacro:macro>
 <joint name="base_footprint_joint" type="fixed">
-    	<origin xyz="0.0 0.0 ${wheel_radius}" rpy="0.0 0.0 0.0"/>
+    	<origin xyz="0.0 0.0 0.08" rpy="0.0 0.0 0.0"/>  <!-- 8cm từ đáy thân xuống mặt đất -->
         <parent link="base_footprint"/>
         <child link="base_link"/>
@@ -104,5 +104,5 @@
         <parent link="base_link"/>
         <child link="post_fl"/>
-        <origin xyz="0.15 -0.2 0.15"/>
+        <origin xyz="0.14 -0.20 0.20"/>  <!-- Góc trước trái, tâm cao 20cm (0-40cm cao) -->
     </joint>
     <link name="post_fl">
@@ -129,5 +129,5 @@
         <parent link="base_link"/>
         <child link="post_fr"/>
-        <origin xyz="0.15 0.2 0.15"/>
+        <origin xyz="0.14 0.20 0.20"/>  <!-- Góc trước phải, tâm cao 20cm (0-40cm cao) -->
     </joint>
     <link name="post_fr">
@@ -154,5 +154,5 @@
         <parent link="base_link"/>
         <child link="post_bl"/>
-        <origin xyz="-0.15 -0.2 0.15"/>
+        <origin xyz="-0.14 -0.20 0.20"/>  <!-- Góc sau trái, tâm cao 20cm (0-40cm cao) -->
     </joint>
     <link name="post_bl">
@@ -179,5 +179,5 @@
         <parent link="base_link"/>
         <child link="post_br"/>
-        <origin xyz="-0.15 0.2 0.15"/>
+        <origin xyz="-0.14 0.20 0.20"/>  <!-- Góc sau phải, tâm cao 20cm (0-40cm cao) -->
     </joint>
     <link name="post_br">
@@ -204,5 +204,5 @@
         <parent link="base_link"/>
         <child link="layer_middle"/>
-        <origin xyz="0.0 0.0 0.15" rpy="0.0 0.0 0.0"/>
+        <origin xyz="0.0 0.0 0.07" rpy="0.0 0.0 0.0"/>  <!-- 7cm từ đáy thân -->
     </joint>
     <link name="layer_middle">
@@ -229,5 +229,5 @@
         <parent link="base_link"/>
         <child link="layer_top"/>
-        <origin xyz="0.0 0.0 0.295" rpy="0.0 0.0 0.0"/>
+        <origin xyz="0.0 0.0 0.33" rpy="0.0 0.0 0.0"/>  <!-- 33cm từ đáy thân -->
     </joint>
     <link name="layer_top">
@@ -300,10 +300,10 @@
 		<parent link="base_link"/>
 		<child link="caster_wheel"/>
-		<origin xyz="-0.1 0.0 -0.022"/>
+		<origin xyz="-0.11 0.0 -0.035"/>  <!-- Caster wheel: 11cm phía sau tâm, từ đáy thân 8cm + 1.5cm bán kính -->
 	</joint>
 	<link name="caster_wheel">
 		<visual>
 			<geometry>
-				<sphere radius="0.03"/>
+				<sphere radius="0.015"/>  <!-- 1.5cm radius = 3cm đường kính -->
 			</geometry>
 			<material name="red"/>
@@ -311,5 +311,5 @@
 		<collision>
 			<geometry>
-				<sphere radius="0.03"/>
+				<sphere radius="0.015"/>
 			</geometry>
 		</collision>
@@ -320,5 +320,5 @@
 	</link>
 <joint name="joint_scan" type="fixed">
-		<origin xyz="0.0 0.0 0.4" rpy="0 0 ${PI}"/>
+		<origin xyz="0.0 0.0 0.435" rpy="0 0 ${PI}"/>  <!-- LiDAR: 43.5cm từ đáy thân, trung tâm -->
 		<parent link="base_link"/>
 		<child link="laser"/>
@@ -345,5 +345,5 @@
         <parent link="base_link"/>
         <child link="zed2_camera_link"/>
-        <origin xyz="0.15 0.0 0.35" rpy="0 0 0"/>
+        <origin xyz="0.13 0.0 0.455" rpy="0 0 0"/>  <!-- ZED2: 45.5cm từ đáy, 13cm cách tâm về phía trước -->
     </joint>
 </robot>

Commit message: feat: remove zed2 and and urdf d435i

File: src/descriptions/model/wheeled/urdf/mobile_robot.xacro (robot description, xacro)
@@ -338,12 +338,7 @@
         </inertial>
     </link>
-    <xacro:include filename="$(find zed_wrapper)/urdf/zed_macro.urdf.xacro" />
-    <xacro:zed_camera name="zed2" model="zed2" enable_gnss="false">
-        <origin xyz="0 0 0" rpy="0 0 0"/>
-    </xacro:zed_camera>
-    <joint name="zed2_base_joint" type="fixed">
-        <parent link="base_link"/>
-        <child link="zed2_camera_link"/>
-        <origin xyz="0.13 0.0 0.455" rpy="0 0 0"/>  <!-- ZED2: 45.5cm từ đáy, 13cm cách tâm về phía trước -->
-    </joint>
+    <xacro:include filename="$(find realsense2_description)/urdf/_d435i.urdf.xacro"/>
+    <xacro:sensor_d435i parent="base_link" name="camera" use_nominal_extrinsics="true">
+        <origin xyz="0.13 0.0 0.455" rpy="0 0 0"/>
+    </xacro:sensor_d435i>
 </robot>

Commit message: feat:initial camera success

File: src/descriptions/model/wheeled/urdf/mobile_robot.xacro (robot description, xacro)
@@ -340,5 +340,5 @@
     <xacro:include filename="$(find realsense2_description)/urdf/_d435i.urdf.xacro"/>
     <xacro:sensor_d435i parent="base_link" name="camera" use_nominal_extrinsics="true">
-        <origin xyz="0.13 0.0 0.455" rpy="0 0 0"/>
+        <origin xyz="0.09715 0.0 0.405" rpy="0 0 0"/>
     </xacro:sensor_d435i>
 </robot>
